Commit message: live position from gripper

File: ssg48_gripper_description/urdf/ssg48_gripper.urdf.xacro (robot description, xacro)
@@ -89,5 +89,5 @@
     type="prismatic">
     <origin
-      xyz="0 0.039 0.07435"
+      xyz="0 0.015 0.07435"
       rpy="0 0 0" />
     <parent
@@ -96,5 +96,5 @@
       link="left_gripper_finger_link" />
     <axis
-      xyz="0 -1 0" />
+      xyz="0 1 0" />
     <limit
       lower="0"
@@ -146,6 +146,9 @@
     name="right_gripper_finger_joint"
     type="prismatic">
+    <!-- <origin
+      xyz="0 -0.039 0.07435"
+      rpy="0 0 0" /> -->
     <origin
-      xyz="0 -0.039 0.07435"
+      xyz="0 -0.015 0.07435"
       rpy="0 0 0" />
     <parent
@@ -154,5 +157,5 @@
       link="right_gripper_finger_link" />
     <axis
-      xyz="0 1 0" />
+      xyz="0 -1 0" />
     <limit
       lower="0"

Commit message: grasp works

File: ssg48_gripper_description/urdf/ssg48_gripper.urdf.xacro (robot description, xacro)
@@ -3,6 +3,6 @@
      Commit Version: 1.6.0-4-g7f85cfe  Build Version: 1.6.7995.38578
      For more information, please see http://wiki.ros.org/sw_urdf_exporter -->
-<robot
-  name="ssg48_gripper" xmlns:xacro="http://www.ros.org/wiki/xacro">
+<robot name="ssg48_gripper" xmlns:xacro="http://www.ros.org/wiki/xacro">
+  <xacro:macro name="ssg48_gripper">
   <link
     name="gripper_base_link">
@@ -168,3 +168,4 @@
       offset="0" />
   </joint>
+  </xacro:macro>
 </robot>

File: ssg48_gripper_description/urdf/standard_gripper_finger.urdf.xacro (robot description, xacro)
@@ -3,8 +3,8 @@
      Commit Version: 1.6.0-4-g7f85cfe  Build Version: 1.6.7995.38578
      For more information, please see http://wiki.ros.org/sw_urdf_exporter -->
-<robot
-  name="standard gripper finger assmebly urdf">
+<robot name="standard_gripper_finger" xmlns:xacro="http://www.ros.org/wiki/xacro">
+  <xacro:macro name="standard_gripper_finger" params="finger_prefix parent_link *origin">
   <link
-    name="gripper_finger_link">
+    name="${finger_prefix}gripper_finger_link">
     <inertial>
       <origin
@@ -27,5 +27,5 @@
       <geometry>
         <mesh
-          filename="package://standard gripper finger assmebly urdf/meshes/gripper_finger_link.STL" />
+          filename="package://ssg48_gripper_description/meshes/gripper_finger_link.STL" />
       </geometry>
       <material
@@ -41,7 +41,14 @@
       <geometry>
         <mesh
-          filename="package://standard gripper finger assmebly urdf/meshes/gripper_finger_link.STL" />
+          filename="package://ssg48_gripper_description/meshes/gripper_finger_link.STL" />
       </geometry>
     </collision>
   </link>
+  <joint name="${finger_prefix}gripper_finger_interface" type="fixed">
+      <xacro:insert_block name="origin" />
+      <parent link="${parent_link}" />
+      <child link="${finger_prefix}gripper_finger_link" />
+      <!-- <origin xyz="0 0 0" rpy="0 0 0" /> -->
+    </joint>
+  </xacro:macro>
 </robot>
