Commit message: standar gripper fingers

File: ssg48_gripper_description/urdf/adaptive_gripper_finger.xacro (robot description, xacro)
@@ -3,8 +3,8 @@
      Commit Version: 1.6.0-4-g7f85cfe  Build Version: 1.6.7995.38578
      For more information, please see http://wiki.ros.org/sw_urdf_exporter -->
-<robot
-  name="gripper-finger-urdf">
+<robot name="adaptive_gripper_finger" xmlns:xacro="http://www.ros.org/wiki/xacro">
+  <xacro:macro name="adaptive_gripper_finger" params="finger_prefix parent_link *origin" >
   <link
-    name="gripper_finger_link">
+    name="${finger_prefix}gripper_finger">
     <inertial>
       <origin
@@ -27,5 +27,5 @@
       <geometry>
         <mesh
-          filename="package://gripper-finger-urdf/meshes/gripper_finger_link.STL" />
+          filename="package://ssg48_gripper_description/meshes/adaptive_gripper_finger_link.STL" />
       </geometry>
       <material
@@ -41,7 +41,14 @@
       <geometry>
         <mesh
-          filename="package://gripper-finger-urdf/meshes/gripper_finger_link.STL" />
+          filename="package://ssg48_gripper_description/meshes/adaptive_gripper_finger_link.STL" />
       </geometry>
     </collision>
   </link>
+  <joint name="${finger_prefix}gripper_finger_interface" type="fixed">
+      <xacro:insert_block name="origin" />
+      <parent link="${parent_link}" />
+      <child link="${finger_prefix}gripper_finger" />
+      <!-- <origin xyz="0 0 0" rpy="0 0 0" /> -->
+    </joint>
+  </xacro:macro>
 </robot>

File: ssg48_gripper_description/urdf/ssg48.urdf.xacro (robot description, xacro)
@@ -1,21 +1,25 @@
 <?xml version="1.0" encoding="utf-8"?>
     <robot xmlns:xacro="http://www.ros.org/wiki/xacro" name="gripper">
+        <xacro:arg name="standard_fingers" default='False' />
         <!-- <xacro:include filename="$(find ssg48_gripper_description)/urdf/ssg48_gripper.urdf.xacro" /> -->
         <xacro:include filename="ssg48_gripper.xacro" />
         <xacro:ssg48_gripper prefix=""/>
-        <xacro:include filename="standard_gripper_finger.xacro" />
-        <xacro:standard_gripper_finger finger_prefix="left_" parent_link="left_gripper_finger_link">
-                    <origin xyz="0.0 0.0 0.0" rpy="0 0 -1.57"/>
-        </xacro:standard_gripper_finger>
-        <xacro:standard_gripper_finger finger_prefix="right_" parent_link="right_gripper_finger_link">
-                <origin xyz="0.0 0.0 0.0" rpy="0 0 1.57"/>
-        </xacro:standard_gripper_finger>
-<!--
-        <xacro:include filename="standard_gripper_finger.xacro" />
-        <xacro:standard_gripper_finger finger_prefix="left" parent_link="world">
-            <origin xyz="0.0 0.0 0.0" rpy="0 0 0.0"/>
-        </xacro:standard_gripper_finger> -->
-    <!-- <xacro:standard_gripper_finger finger_prefix="right" parent_link="right_gripper_finger_link">
-		<origin xyz="0.0 0.0 3.14" rpy="0 0 0.0"/>
-	</xacro:standard_gripper_finger> -->
+        <xacro:if value="$(arg standard_fingers)">
+                <xacro:include filename="adaptive_gripper_finger.xacro" />
+                <xacro:standard_gripper_finger finger_prefix="left_" parent_link="left_gripper_finger_link">
+                            <origin xyz="0.0 0.0 0.0" rpy="0 0 -1.57"/>
+                </xacro:standard_gripper_finger>
+                <xacro:standard_gripper_finger finger_prefix="right_" parent_link="right_gripper_finger_link">
+                        <origin xyz="0.0 0.0 0.0" rpy="0 0 1.57"/>
+                </xacro:standard_gripper_finger>
+        </xacro:if>
+        <xacro:unless value="$(arg standard_fingers)">
+                <xacro:include filename="adaptive_gripper_finger.xacro" />
+                <xacro:adaptive_gripper_finger finger_prefix="left_" parent_link="left_gripper_finger_link">
+                            <origin xyz="0.0 0.0 0.0" rpy="0 0 -1.57"/>
+                </xacro:adaptive_gripper_finger>
+                <xacro:adaptive_gripper_finger finger_prefix="right_" parent_link="right_gripper_finger_link">
+                        <origin xyz="0.0 0.0 0.0" rpy="0 0 1.57"/>
+                </xacro:adaptive_gripper_finger>
+        </xacro:unless>
     </robot>
