Commit message: a

File: ssg48_gripper_description/urdf/ssg48.urdf.xacro (robot description, xacro)
@@ -1,9 +1,9 @@
 <?xml version="1.0" encoding="utf-8"?>
-    <robot name="gripper" xmlns:xacro="http://www.ros.org/wiki/xacro">
+    <robot xmlns:xacro="http://www.ros.org/wiki/xacro" name="gripper">
         <link name="world"/>
         <!-- <xacro:include filename="$(find ssg48_gripper_description)/urdf/ssg48_gripper.urdf.xacro" /> -->
-        <!-- <xacro:include filename="$(find ssg48_gripper_description)/urdf/ssg48.urdf.xacro" />
-        <xacro:ssg48_gripper/> -->
-        <xacro:include filename="$(find ssg48_gripper_description)/urdf/standard_gripper_finger.urdf.xacro" />
+        <!-- <xacro:include filename="ssg48_gripper.xacro" /> -->
+        <!-- <xacro:ssg48_gripper/> -->
+        <xacro:include filename="standard_gripper_finger.xacro" />
         <xacro:standard_gripper_finger finger_prefix="left" parent_link="world">
             <origin xyz="0.0 0.0 0.0" rpy="0 0 0.0"/>

File: ssg48_gripper_description/urdf/ssg48_gripper.urdf.xacro (robot description, xacro)
@@ -4,5 +4,5 @@
      For more information, please see http://wiki.ros.org/sw_urdf_exporter -->
 <robot name="ssg48_gripper" xmlns:xacro="http://www.ros.org/wiki/xacro">
-  <xacro:macro name="ssg48_gripper">
+  <!-- <xacro:macro name="ssg48_gripper"> -->
   <link
     name="gripper_base_link">
@@ -168,4 +168,4 @@
       offset="0" />
   </joint>
-  </xacro:macro>
+  <!-- </xacro:macro> -->
 </robot>

File: ssg48_gripper_description/urdf/standard_gripper_finger.xacro (robot description, xacro)
@@ -1,8 +1,5 @@
-<?xml version="1.0" encoding="utf-8"?>
-<!-- This URDF was automatically created by SolidWorks to URDF Exporter! Originally created by Stephen Brawner (brawner@gmail.com)
-     Commit Version: 1.6.0-4-g7f85cfe  Build Version: 1.6.7995.38578
-     For more information, please see http://wiki.ros.org/sw_urdf_exporter -->
+<?xml version="1.0"?>
 <robot name="standard_gripper_finger" xmlns:xacro="http://www.ros.org/wiki/xacro">
-  <xacro:macro name="standard_gripper_finger" params="finger_prefix parent_link *origin">
+  <xacro:macro name="standard_gripper_finger" params="finger_prefix parent_link *origin" >
   <link
     name="${finger_prefix}gripper_finger_link">

Commit message: xacro works better

File: ssg48_gripper_description/urdf/ssg48.urdf.xacro (robot description, xacro)
@@ -1,12 +1,19 @@
 <?xml version="1.0" encoding="utf-8"?>
     <robot xmlns:xacro="http://www.ros.org/wiki/xacro" name="gripper">
-        <link name="world"/>
         <!-- <xacro:include filename="$(find ssg48_gripper_description)/urdf/ssg48_gripper.urdf.xacro" /> -->
-        <!-- <xacro:include filename="ssg48_gripper.xacro" /> -->
-        <!-- <xacro:ssg48_gripper/> -->
+        <xacro:include filename="ssg48_gripper.xacro" />
+        <xacro:ssg48_gripper prefix=""/>
+        <xacro:include filename="standard_gripper_finger.xacro" />
+        <xacro:standard_gripper_finger finger_prefix="left_" parent_link="left_gripper_finger_link">
+                    <origin xyz="0.0 0.0 0.0" rpy="0 0 -1.57"/>
+        </xacro:standard_gripper_finger>
+        <xacro:standard_gripper_finger finger_prefix="right_" parent_link="right_gripper_finger_link">
+                <origin xyz="0.0 0.0 0.0" rpy="0 0 1.57"/>
+        </xacro:standard_gripper_finger>
+<!--
         <xacro:include filename="standard_gripper_finger.xacro" />
         <xacro:standard_gripper_finger finger_prefix="left" parent_link="world">
             <origin xyz="0.0 0.0 0.0" rpy="0 0 0.0"/>
-        </xacro:standard_gripper_finger>
+        </xacro:standard_gripper_finger> -->
     <!-- <xacro:standard_gripper_finger finger_prefix="right" parent_link="right_gripper_finger_link">
 		<origin xyz="0.0 0.0 3.14" rpy="0 0 0.0"/>

File: ssg48_gripper_description/urdf/ssg48_gripper.xacro (robot description, xacro)
@@ -4,5 +4,5 @@
      For more information, please see http://wiki.ros.org/sw_urdf_exporter -->
 <robot name="ssg48_gripper" xmlns:xacro="http://www.ros.org/wiki/xacro">
-  <!-- <xacro:macro name="ssg48_gripper"> -->
+  <xacro:macro name="ssg48_gripper" params="prefix" >
   <link
     name="gripper_base_link">
@@ -168,4 +168,4 @@
       offset="0" />
   </joint>
-  <!-- </xacro:macro> -->
+  </xacro:macro>
 </robot>

File: ssg48_gripper_description/urdf/standard_gripper_finger.xacro (robot description, xacro)
@@ -3,5 +3,5 @@
   <xacro:macro name="standard_gripper_finger" params="finger_prefix parent_link *origin" >
   <link
-    name="${finger_prefix}gripper_finger_link">
+    name="${finger_prefix}gripper_finger">
     <inertial>
       <origin
@@ -24,5 +24,5 @@
       <geometry>
         <mesh
-          filename="package://ssg48_gripper_description/meshes/gripper_finger_link.STL" />
+          filename="package://ssg48_gripper_description/meshes/standard_gripper_finger_link.STL" />
       </geometry>
       <material
@@ -38,5 +38,5 @@
       <geometry>
         <mesh
-          filename="package://ssg48_gripper_description/meshes/gripper_finger_link.STL" />
+          filename="package://ssg48_gripper_description/meshes/standard_gripper_finger_link.STL" />
       </geometry>
     </collision>
@@ -45,5 +45,5 @@
       <xacro:insert_block name="origin" />
       <parent link="${parent_link}" />
-      <child link="${finger_prefix}gripper_finger_link" />
+      <child link="${finger_prefix}gripper_finger" />
       <!-- <origin xyz="0 0 0" rpy="0 0 0" /> -->
     </joint>

Commit message: adaptive finger

File: ssg48_gripper_description/urdf/ssg48.urdf.xacro (robot description, xacro)
@@ -1,5 +1,5 @@
 <?xml version="1.0" encoding="utf-8"?>
     <robot xmlns:xacro="http://www.ros.org/wiki/xacro" name="gripper">
-        <xacro:arg name="standard_fingers" default='False' />
+        <xacro:arg name="standard_fingers" default='True' />
         <!-- <xacro:include filename="$(find ssg48_gripper_description)/urdf/ssg48_gripper.urdf.xacro" /> -->
         <xacro:include filename="ssg48_gripper.xacro" />
@@ -17,8 +17,8 @@
                 <xacro:include filename="adaptive_gripper_finger.xacro" />
                 <xacro:adaptive_gripper_finger finger_prefix="left_" parent_link="left_gripper_finger_link">
-                            <origin xyz="0.0 0.0 0.0" rpy="0 0 -1.57"/>
+                            <origin xyz="0.0 0.0 0.0" rpy="0 -1.57 -3.14"/>
                 </xacro:adaptive_gripper_finger>
                 <xacro:adaptive_gripper_finger finger_prefix="right_" parent_link="right_gripper_finger_link">
-                        <origin xyz="0.0 0.0 0.0" rpy="0 0 1.57"/>
+                        <origin xyz="0.0 0.0 0.0" rpy="0 -1.57 0"/>
                 </xacro:adaptive_gripper_finger>
         </xacro:unless>

Commit message: urdf update

File: ssg48_gripper_description/urdf/ssg48.urdf.xacro (robot description, xacro)
@@ -1,10 +1,13 @@
 <?xml version="1.0" encoding="utf-8"?>
     <robot xmlns:xacro="http://www.ros.org/wiki/xacro" name="gripper">
+        <link name="world" />
         <xacro:arg name="standard_fingers" default='True' />
         <!-- <xacro:include filename="$(find ssg48_gripper_description)/urdf/ssg48_gripper.urdf.xacro" /> -->
         <xacro:include filename="ssg48_gripper.xacro" />
-        <xacro:ssg48_gripper prefix=""/>
+        <xacro:ssg48_gripper prefix="" parent_link="world">
+                            <origin xyz="0.0 0.0 0.0" rpy="0 0 0"/>
+                </xacro:ssg48_gripper>
         <xacro:if value="$(arg standard_fingers)">
-                <xacro:include filename="adaptive_gripper_finger.xacro" />
+                <xacro:include filename="standard_gripper_finger.xacro" />
                 <xacro:standard_gripper_finger finger_prefix="left_" parent_link="left_gripper_finger_link">
                             <origin xyz="0.0 0.0 0.0" rpy="0 0 -1.57"/>

File: ssg48_gripper_description/urdf/ssg48_gripper.xacro (robot description, xacro)
@@ -4,7 +4,7 @@
      For more information, please see http://wiki.ros.org/sw_urdf_exporter -->
 <robot name="ssg48_gripper" xmlns:xacro="http://www.ros.org/wiki/xacro">
-  <xacro:macro name="ssg48_gripper" params="prefix" >
+  <xacro:macro name="ssg48_gripper" params="prefix parent_link *origin" >
   <link
-    name="gripper_base_link">
+    name="${prefix}gripper_base_link">
     <inertial>
       <origin
@@ -46,5 +46,5 @@
   </link>
   <link
-    name="left_gripper_finger_link">
+    name="${prefix}left_gripper_finger_link">
     <inertial>
       <origin
@@ -86,5 +86,5 @@
   </link>
   <joint
-    name="left_gripper_finger_joint"
+    name="${prefix}left_gripper_finger_joint"
     type="prismatic">
     <origin
@@ -92,7 +92,7 @@
       rpy="0 0 0" />
     <parent
-      link="gripper_base_link" />
+      link="${prefix}gripper_base_link" />
     <child
-      link="left_gripper_finger_link" />
+      link="${prefix}left_gripper_finger_link" />
     <axis
       xyz="0 1 0" />
@@ -104,5 +104,5 @@
   </joint>
   <link
-    name="right_gripper_finger_link">
+    name="${prefix}right_gripper_finger_link">
     <inertial>
       <origin
@@ -144,5 +144,5 @@
   </link>
   <joint
-    name="right_gripper_finger_joint"
+    name="${prefix}right_gripper_finger_joint"
     type="prismatic">
     <!-- <origin
@@ -153,7 +153,7 @@
       rpy="0 0 0" />
     <parent
-      link="gripper_base_link" />
+      link="${prefix}gripper_base_link" />
     <child
-      link="right_gripper_finger_link" />
+      link="${prefix}right_gripper_finger_link" />
     <axis
       xyz="0 -1 0" />
@@ -164,8 +164,14 @@
       velocity="1" />
     <mimic
-      joint="left_gripper_finger_joint"
+      joint="${prefix}left_gripper_finger_joint"
       multiplier="1"
       offset="0" />
   </joint>
+  <joint name="${prefix}gripper_interface" type="fixed">
+      <xacro:insert_block name="origin" />
+      <parent link="${parent_link}" />
+      <child link="${prefix}gripper_base_link" />
+      <!-- <origin xyz="0 0 0" rpy="0 0 0" /> -->
+    </joint>
   </xacro:macro>
 </robot>

Commit message: tcp

File: ssg48_gripper_description/urdf/ssg48.urdf.xacro (robot description, xacro)
@@ -5,8 +5,9 @@
         <!-- <xacro:include filename="$(find ssg48_gripper_description)/urdf/ssg48_gripper.urdf.xacro" /> -->
         <xacro:include filename="ssg48_gripper.xacro" />
-        <xacro:ssg48_gripper prefix="" parent_link="world">
+        <xacro:if value="$(arg standard_fingers)">
+                <xacro:ssg48_gripper prefix="" parent_link="world" gripper_finger_tcp="0.031">
                             <origin xyz="0.0 0.0 0.0" rpy="0 0 0"/>
+                            <!-- <gripper_tcp xyz="0.0 0.0 ${0.07435+0.031}" rpy="0 0 0"/> -->
                 </xacro:ssg48_gripper>
-        <xacro:if value="$(arg standard_fingers)">
                 <xacro:include filename="standard_gripper_finger.xacro" />
                 <xacro:standard_gripper_finger finger_prefix="left_" parent_link="left_gripper_finger_link">
@@ -18,4 +19,8 @@
         </xacro:if>
         <xacro:unless value="$(arg standard_fingers)">
+                <xacro:ssg48_gripper prefix="" parent_link="world" gripper_finger_tcp="0.070">
+                            <origin xyz="0.0 0.0 0.0" rpy="0 0 0"/>
+                            <!-- <gripper_tcp xyz="0.0 0.0 ${0.07435+0.070}" rpy="0 0 0"/> -->
+                </xacro:ssg48_gripper>
                 <xacro:include filename="adaptive_gripper_finger.xacro" />
                 <xacro:adaptive_gripper_finger finger_prefix="left_" parent_link="left_gripper_finger_link">

File: ssg48_gripper_description/urdf/ssg48_gripper.xacro (robot description, xacro)
@@ -4,5 +4,5 @@
      For more information, please see http://wiki.ros.org/sw_urdf_exporter -->
 <robot name="ssg48_gripper" xmlns:xacro="http://www.ros.org/wiki/xacro">
-  <xacro:macro name="ssg48_gripper" params="prefix parent_link *origin" >
+  <xacro:macro name="ssg48_gripper" params="prefix parent_link *origin gripper_finger_tcp:=0.031" >
   <link
     name="${prefix}gripper_base_link">
@@ -174,4 +174,13 @@
       <!-- <origin xyz="0 0 0" rpy="0 0 0" /> -->
     </joint>
+    <link
+    name="${prefix}gripper_tcp_link">
+  </link>
+  <joint name="${prefix}gripper_tcp_joint" type="fixed">
+      <parent link="${prefix}gripper_base_link" />
+      <child link="${prefix}gripper_tcp_link" />
+      <!-- <xacro:insert_block name="gripper_tcp" /> -->
+      <origin xyz="0 0 ${gripper_finger_tcp+0.07435}" rpy="0 0 0" />
+    </joint>
   </xacro:macro>
 </robot>
