Commit message: define tcp self

File: ssg48_gripper_description/urdf/ssg48_gripper.xacro (robot description, xacro)
@@ -174,13 +174,12 @@
       <!-- <origin xyz="0 0 0" rpy="0 0 0" /> -->
     </joint>
-    <link
+    <!-- <link
     name="${prefix}gripper_tcp_link">
-  </link>
-  <joint name="${prefix}gripper_tcp_joint" type="fixed">
+  </link> -->
+  <!-- <joint name="${prefix}gripper_tcp_joint" type="fixed">
       <parent link="${prefix}gripper_base_link" />
       <child link="${prefix}gripper_tcp_link" />
-      <!-- <xacro:insert_block name="gripper_tcp" /> -->
       <origin xyz="0 0 ${gripper_finger_tcp+0.07435}" rpy="0 0 0" />
-    </joint>
+    </joint> -->
   </xacro:macro>
 </robot>
